Commit message: More progress

File: urdf/edukit_bot.urdf (robot description, URDF)
Before this commit: robot edukit_bot, 4 links, 3 joints
Links:
- removed link left_wheel
- removed link right_wheel
- added link wheel_left; visual cylinder length=0.025 radius=0.032
- added link wheel_right; visual cylinder length=0.025 radius=0.032
Joints:
- removed joint left_wheel_joint
- removed joint right_wheel_joint
- added joint wheel_left_joint: type continuous, parent base_link, child wheel_left, origin xyz=0.056 -0.058 0 rpy=0 0 0, axis 0 1 0
- added joint wheel_right_joint: type continuous, parent base_link, child wheel_right, origin xyz=0.056 0.058 0 rpy=0 0 0, axis 0 1 0
